File: teensy40-bb-hc05-adapter/teensy40-bb-hc05-adapter.kicad_pcb (KiCad board)
At the start: 2 copper layers, 18 x 71.6 mm, 17 parts, among them J1 Conn_01x06_0.1_Header, J2 Conn_01x06_0.1_Socket, J3 Conn_01x08, J4 Conn_01x08, U1 74LVC1G17, U2 74LVC1G14, U3 Teensy4.0_WithBottomAndEdge

Commit message: Revise routing
Routing:
- net GND: track 7.34 -> 6.41 mm
- net +5V: track 50.6 -> 50.1 mm
Other:
- board text added: "CTS"
- board text added: "FTDI"
- board text added: "HC-05"
- board text added: "HC-05 Arduino Programming Adapter"
- board text removed: "JLCJLCJLCJLC"

Commit message: Clean up positions
Parts:
- moved U1 0.64 mm to (135.9, 136.1)
- moved U2 0.64 mm to (135.9, 141.2)
- moved C3 0.63 mm to (131.4, 141.2)
- moved R3 0.63 mm to (131.4, 136.1)
Routing:
- net Net-(R3-Pad2): track 3.13 -> 4.40 mm
- net GND: track 6.41 -> 5.69 mm
Other:
- board text added: "RXI"
- board text added: "RXO"
- board text added: "TXI"
- board text added: "TXO"
- board text removed: "RX"
- board text removed: "TX"

Commit message: Clean up more
Parts:
- added REF**: OSHW-Logo2_7.3x6mm_SilkScreen, Symbol:OSHW-Logo2_7.3x6mm_SilkScreen, B.Cu at (134.6, 116.8)
Other:
- board text added: "RX"
- board text added: "RXD"
- board text added: "TX"
- board text added: "TXD"
- board text removed: "RXI"
- board text removed: "RXO"
- board text removed: "TXI"
- board text removed: "TXO"

Commit message: Add more silkscreen labels
Parts:
- moved J1 35.9 mm to (101.6, 106.9)
- moved J2 35.9 mm to (116.8, 106.9)
- moved J3 35.9 mm to (101.6, 86.4)
- moved J4 35.9 mm to (116.8, 86.4)
- moved REF** 35.9 mm to (109.2, 91.4) (x2)
- moved U3 35.9 mm to (109.2, 50.8)
- moved C1 35.9 mm to (109.2, 109.5)
- moved C2 35.9 mm to (109.2, 117.1)
- moved JP1 35.9 mm to (106.0, 106.9)
- moved JP2 35.9 mm to (106.0, 119.6)
- moved R1 35.9 mm to (107.3, 113.3)
- moved R2 35.9 mm to (111.1, 113.3)
- moved R3 35.9 mm to (106.0, 110.7)
- moved U1 35.9 mm to (110.5, 110.7)
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